File: _MK3_/PCB/MK3_v1.5/Mechanics.kicad_sch (KiCad schematic)
At the start: 8 parts, among them SW3 SW_DPDT_x2

Commit message: PCB UPDATE
Connections:
- net VBus_USB: now reaches TP4.1
Changed lines of the file:
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@@
+	(wire
+		(pts
+			(xy 161.29 35.56) (xy 161.29 34.29)
+		)
+		(stroke
+			(width 0)
+			(type default)
+		)
+	)
 	(wire
 		(pts
@@
 			(effects
 				(font
+					(size 1.27 1.27)
+				)
+				(justify right)
+				(hide yes)
+			)
+		)
+	)
+	(global_label "VBus_USB"
+		(shape input)
+		(at 161.29 35.56 270)
+		(fields_autoplaced yes)
+		(effects
+			(font
+				(size 1.27 1.27)
+			)
+			(justify right)
+		)
+		(property "Intersheetrefs" "${INTERSHEET_REFS}"
+			(at 161.29 46.5614 90)
+			(effects
+				(font
