File: _MK3_/PCB/MK3_v1.5/MK3_v1.5.kicad_pcb (KiCad board)
At the start: 2 copper layers, 95 x 60 mm, 87 parts, among them IC1 DRV8874PWPR, IC2 DRV8874PWPR, IC3 TPS565242DRLR, J1 XT30PW-M, J10 Conn_01x04_Pin, J11 USB_TypeC, J2 Conn_01x06_Pin, J3 Conn_01x06_Pin, J4 Conn_01x06_Pin, J5 Conn_01x03_Pin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

Commit message: PCB UPDATE
Parts:
- added L1: 3.3uH, Inductor_SMD:L_Vishay_IHLP-1616, F.Cu at (188.9, 96.6)
- added L2: 1.5uH, Inductor_SMD:L_Vishay_IHLP-1212, F.Cu at (184.6, 78.3)
- C17, R10, R15: moved to B.Cu
- moved R6 159.4 mm to (184.8, 100.5), turned to 180 degrees
- moved U2 159.3 mm to (185.4, 96.5), turned to 180 degrees
- moved IC3 159.2 mm to (185.3, 81.3), turned to -90 degrees
- moved R11 157.1 mm to (188.1, 83.7)
- moved R7 155.5 mm to (181.1, 100.5), turned to 180 degrees
- moved C5 155.3 mm to (189.2, 102.8), turned to 180 degrees
- moved C6 154.4 mm to (189.2, 100.8), turned to 180 degrees
- moved R12 154.2 mm to (185.2, 84.6), turned to 90 degrees
- moved C11 152.2 mm to (188.8, 81.2)
- moved R8 151.8 mm to (181.0, 94.7)
- moved R9 151.6 mm to (181.0, 96.5), turned to 180 degrees
- moved C3 150.2 mm to (184.2, 98.5), turned to 180 degrees
- moved C12 146.9 mm to (188.8, 79.1)
- moved C16 145.4 mm to (181.8, 81.2), turned to 180 degrees
- moved C15 145.2 mm to (181.8, 83.3), turned to 180 degrees
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Connections:
- TP4 pad 1: unconnected-(TP4-Pad1) -> VBus_USB
Routing:
- net +3V3: track 60.5 -> 179.3 mm, vias 0 -> 3
- net +5V: track 62.6 -> 130.7 mm, vias 5 -> 7
- net +12V: track 74.3 -> 92.5 mm
- net Vout_5V: track 2.69 -> 20.5 mm, vias 0 -> 2
- net Net-(U2-EN): track 0.00 -> 7.36 mm, vias 0 -> 2
- net Net-(U2-FB): track 0.00 -> 5.05 mm
- net GND: track 33.1 -> 38.1 mm, vias 20 -> 22
- net FB: track 0.00 -> 3.98 mm
- net Net-(C17-Pad2): track 0.00 -> 3.53 mm
- net Net-(U2-SW): track 0.00 -> 3.25 mm
- net VBus_USB: track 12.7 -> 16.0 mm
- net Net-(U2-BST): track 0.00 -> 1.99 mm
- net EN: track 29.4 -> 30.3 mm
Other:
- board text added: "VUSB"

Commit message: pcb done
Parts:
- removed D5: LED, LED_SMD:LED_0805_2012Metric_Pad1.15x1.40mm_HandSolder
- removed R5: R, Resistor_SMD:R_0805_2012Metric_Pad1.20x1.40mm_HandSolder
- R16: moved to B.Cu
- moved TP3 46.6 mm to (176.5, 91.3)
- moved R16 13.6 mm to (125.2, 87.6)
- moved C11 3.84 mm to (188.8, 85.0)
- moved C12 3.84 mm to (188.8, 83.0)
- moved C13 3.84 mm to (181.8, 89.2)
- moved C14 3.84 mm to (182.2, 91.3)
- moved C16 3.84 mm to (181.8, 85.0)
- moved IC3 3.84 mm to (185.3, 85.1)
- moved R11 3.84 mm to (188.1, 87.5)
- moved C15 3.84 mm to (181.8, 87.1)
- moved L2 3.84 mm to (184.6, 82.1)
- moved R12 3.84 mm to (185.2, 88.4)
- moved TP4 2.56 mm to (112.3, 110.6)
- moved R21 2.40 mm to (188.7, 105.8)
- moved R22 2.40 mm to (190.7, 105.8)
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Connections:
- IC2 pad 1: EnL -> EnR
- IC2 pad 2: PhL -> PhR
- U1 pad 10: unconnected-(U1-IO17-Pad10) -> SCL
- U1 pad 11: unconnected-(U1-IO18-Pad11) -> SDA
- U1 pad 12: unconnected-(U1-IO8-Pad12) -> SHARP1
- U1 pad 20: unconnected-(U1-IO12-Pad20) -> NFault
- U1 pad 21: unconnected-(U1-IO13-Pad21) -> PhL
- U1 pad 22: unconnected-(U1-IO14-Pad22) -> EnL
- U1 pad 23: unconnected-(U1-IO21-Pad23) -> IR
- U1 pad 24: unconnected-(U1-IO47-Pad24) -> LED2
- U1 pad 25: unconnected-(U1-IO48-Pad25) -> LED1
- U1 pad 38: unconnected-(U1-IO2-Pad38) -> SW2
- U1 pad 39: unconnected-(U1-IO1-Pad39) -> SW1
- U1 pad 4: unconnected-(U1-IO4-Pad4) -> QRE_A
- U1 pad 5: unconnected-(U1-IO5-Pad5) -> QRE_B
- U1 pad 6: unconnected-(U1-IO6-Pad6) -> QRE_C
- U1 pad 7: unconnected-(U1-IO7-Pad7) -> SHARP2
- U1 pad 8: unconnected-(U1-IO15-Pad8) -> EnR
- U1 pad 9: unconnected-(U1-IO16-Pad9) -> PhR
Routing:
- net QRE_B: track 0.00 -> 54.1 mm, vias 0 -> 3
- net QRE_A: track 0.00 -> 51.8 mm, vias 0 -> 1
- net SHARP1: track 0.00 -> 45.5 mm, vias 0 -> 3
- net NFault: track 0.00 -> 44.6 mm, vias 0 -> 3
- net EnR: track 0.00 -> 41.5 mm, vias 0 -> 2
- net PhR: track 0.00 -> 39.6 mm, vias 0 -> 2
- net QRE_C: track 2.75 -> 40.0 mm, vias 0 -> 3
- net SDA: track 39.5 -> 71.3 mm, vias 0 -> 2
- net +3V3: track 179.3 -> 211.1 mm, vias 3 -> 5
- net SCL: track 40.2 -> 71.2 mm, vias 0 -> 1
- net IR: track 0.00 -> 29.6 mm
- net SHARP2: track 0.00 -> 28.0 mm, vias 0 -> 1
- net EnL: track 0.00 -> 16.3 mm
- net PhL: track 0.00 -> 15.9 mm
- net LED2: track 0.00 -> 15.5 mm
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Other:
- board text added: "3V3"
- board text added: "LEDS"
- board text added: "OFF"
- board text added: "ON"
