File: _MK-1_/NeoSumec_MK-1/NeoSumec_MK-1.kicad_sch (KiCad schematic)
At the start: 0 parts

Commit message: .gitignore
Other:
- added sheet Senzors (senzors.kicad_sch)
Changed lines of the file:
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@@
 (kicad_sch
-	(version 20250114)
+	(version 20260306)
 	(generator "eeschema")
-	(generator_version "9.0")
+	(generator_version "10.0")
 	(paper "A4")
+	(sheet
+		(at 21.59 21.59)
+		(size 35.56 29.21)
+		(exclude_from_sim no)
+		(in_bom yes)
+		(on_board yes)
+		(dnp no)
+		(fields_autoplaced yes)
+		(stroke
+			(width 0.1524)
+			(type solid)
+		)
+		(fill
+			(color 0 0 0 0)
+		)
+		(property "Sheetname" "Senzors"
+			(at 21.59 20.8784 0)
+			(show_name no)
+			(do_not_autoplace no)
+			(effects
+				(font
+					(size 1.27 1.27)
+				)
+				(justify left bottom)
+			)
+		)
+		(property "Sheetfile" "senzors.kicad_sch"
+			(at 21.59 51.3846 0)
+			(show_name no)
+			(do_not_autoplace no)
+			(effects
+				(font
+					(size 1.27 1.27)
+				)
+				(justify left top)
+			)
+		)
+		(instances
+			(project "NeoSumec_MK-1"
+				(path "/9e88de0f-3b60-48fb-b244-fba2a5cbc7b8"
+					(page "2")
+				)
+			)
+		)
+	)
 	(sheet_instances
 		(path "/"

Commit message: QRE-BOARD UPDATE
Redesighned QRE-BackSen to maxbe latest eteration for now

Added some changes on mk-1 DPS desighn too (Not that much)
Parts:
- added C1: C, symbol Device:C
- added C10, C4, C7: 100nF, symbol Device:C
- added C11, C5: 10uF, symbol Device:C_Polarized
- added C2: C_Polarized, symbol Device:C_Polarized
- added C3, C9: 100nF, symbol Device:C_Small
- added C6, C8: 22nF, symbol Device:C_Small
- added IC1, IC2: DRV8874PWPR, Package_SO:HTSSOP-16-1EP_4.4x5mm_P0.65mm_EP3.4x5mm_Mask2.46x2.31mm, symbol neo_sumec_symbols:DRV8874PWPR
- added J1, J2, J3, J4, J5, J7, J8: Conn_01x03_Pin, Connector_Molex:Molex_PicoBlade_53398-0371_1x03-1MP_P1.25mm_Vertical, symbol Connector:Conn_01x03_Pin
- added J6: Conn_01x04_Pin, Connector_Molex:Molex_PicoBlade_53398-0471_1x04-1MP_P1.25mm_Vertical, symbol Connector:Conn_01x04_Pin
- added JPL, JPL1: SolderJumper_3_Open, Jumper:SolderJumper-3_P2.0mm_Open_TrianglePad1.0x1.5mm, symbol Jumper:SolderJumper_3_Open
- added R1: 10k, symbol Device:R
- added R2: R, symbol Device:R
- added SWBoot: SW_Push, symbol Switch:SW_Push
- added U1: ESP32-S3-WROOM-1, PCM_Espressif:ESP32-S3-WROOM-1, symbol neo_sumec_symbols:ESP32-S3-WROOM-1_CUSTOM_made_by_bismarx
Connections:
- new net: C6.1, IC1.13 (CPH)
- new net: C6.2, IC1.14 (CPL)
- new net: C3.1, IC1.12 (VCP)
- new net: C8.1, IC2.13 (CPH)
- new net: C8.2, IC2.14 (CPL)
- new net: C9.1, IC2.12 (VCP)
- new net +3.3V: IC1.3 (NSLEEP), IC1.5 (VREF), IC2.3 (NSLEEP), IC2.5 (VREF), J1.2 (Pin_2), J2.2 (Pin_2), J3.2 (Pin_2), J4.2 (Pin_2), J5.2 (Pin_2), J6.2 (Pin_2), J7.2 (Pin_2), J8.1 (Pin_1), JPL.1 (A), JPL1.1 (A), R1.2
- new net Boot: C7.1, SWBoot.1, U1.27 (IO0)
- new net D+: U1.14 (IO20)
- new net D-: U1.13 (IO19)
- new net EN: U1.3 (EN)
- new net ENL: IC1.1 (EN/IN1)
- new net ENR: IC2.1 (EN/IN1)
- new net GND: C10.2, C11.2, C4.2, C5.2, C7.2, IC1.15 (GND), IC1.17 (EP), IC1.6 (IPROPI), IC1.7 (IMODE), IC1.9 (PGND), IC2.15 (GND), IC2.17 (EP), IC2.6 (IPROPI), IC2.7 (IMODE), IC2.9 (PGND), J1.3 (Pin_3), J2.3 (Pin_3), J3.3 (Pin_3), J4.3 (Pin_3), J5.3 (Pin_3), J6.3 (Pin_3), J7.3 (Pin_3), J8.2 (Pin_2), JPL.3 (B), JPL1.3 (B), SWBoot.2, U1.1 (GND), U1.40 (GND), U1.41 (GND)
- new net IR_Sen: J8.3 (Pin_3)
- new net ML1: IC1.8 (OUT1)
- new net ML2: IC1.10 (OUT2)
- new net MR1: IC2.8 (OUT1)
- new net MR2: IC2.10 (OUT2)
- new net PHL: IC1.2 (PH/IN2)
- new net PHR: IC2.2 (PH/IN2)
- new net PMODEL: IC1.16 (PMODE), JPL.2 (C)
- new net PMODER: IC2.16 (PMODE), JPL1.2 (C)
- new net QRE_Back: J7.1 (Pin_1)
- new net QRE_Left: J6.1 (Pin_1)
- new net QRE_Right: J6.4 (Pin_4)
- new net Sharp90Left: J4.1 (Pin_1)
- new net Sharp90Right: J5.1 (Pin_1)
- new net SharpLeft: J1.1 (Pin_1)
- new net SharpMiddle: J2.1 (Pin_1)
- new net SharpRight: J3.1 (Pin_1)
- new net VCC: C10.1, C11.1, C3.2, C4.1, C5.1, C9.2, IC1.11 (VM), IC2.11 (VM)
- new net nFault: IC1.4 (NFAULT), IC2.4 (NFAULT), R1.1
- no-connect marks 0 -> 3
Other:
- removed sheet Senzors
- note added: "EN - High: chip on Low: chip off"
- note added: "ESP32-S3-Wroom-1 Datasheet"
- note added: "IR Sen"
- note added: "Left"
- note added: "QRE Back"
- note added: "QRE front"
- note added: "Right"
- note added: "Sharp front row"
- note added: "Sharp side"
- note added: "TSOP XXXX"
- company: (none) -> RoboCrew - Prosek
- title: (none) -> NeoSumec MK-1
