File: _MK-1_/NeoSumec_MK-1/NeoSumec_MK-1.kicad_sch (KiCad schematic)
At the start: 27 parts, among them IC1 DRV8874PWPR, IC2 DRV8874PWPR, J1 Conn_01x03_Pin, J2 Conn_01x03_Pin, J3 Conn_01x03_Pin, J4 Conn_01x03_Pin, J5 Conn_01x03_Pin, J6 Conn_01x04_Pin, J7 Conn_01x03_Pin, J8 Conn_01x03_Pin, U1 ESP32-S3-WROOM-1

Commit message: MK-1 Designing
Parts:
- J8: footprint Connector_Molex:Molex_PicoBlade_53398-0371_1x03-1MP_P1.25mm_Vertical -> TerminalBlock:TerminalBlock_Xinya_XY308-2.54-3P_1x03_P2.54mm_Horizontal
- renumbered JPL1 to JPR
Other:
- company: RoboCrew - Prosek -> Maded by Vadim Sobčuk
- moved on the sheet: C1, C10, C11, C2, C3, C4, C5, C6, C7, C8, C9, IC1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
