File: _QRE-Board_/QREBoard/QREBoard.kicad_pcb (KiCad board)
At the start: 2 copper layers, 11 parts, among them J1 Conn_01x04_Pin

Commit message: some changes
Parts:
- added H3: M3, MountingHole:MountingHole_3.2mm_M3_Pad_Via, F.Cu at (93.6, 112.3)
- added R5: 100R, Resistor_SMD:R_0805_2012Metric_Pad1.20x1.40mm_HandSolder, F.Cu at (93.6, 104.9)
- added R6: 10K, Resistor_SMD:R_0805_2012Metric_Pad1.20x1.40mm_HandSolder, F.Cu at (92.6, 107.7)
- added S3: QRE1113, OptoDevice:OnSemi_CASE100AQ, F.Cu at (95.6, 104.0)
- moved TP2 1.51 mm to (141.5, 99.7)
Routing:
- net GND: track 0.00 -> 12.1 mm
- net Net-(S3-A): track 0.00 -> 2.04 mm
- net QRE_Back: track 0.00 -> 1.90 mm
- net +3V3: track 0.00 -> 1.80 mm
Other:
- board outline added: 5.9 x 12.7 mm

Commit message: QRE-BOARD UPDATE
Redesighned QRE-BackSen to maxbe latest eteration for now

Added some changes on mk-1 DPS desighn too (Not that much)
Parts:
- H3: footprint MountingHole:MountingHole_3.2mm_M3_Pad_Via -> MountingHole:MountingHole_3.2mm_M3_ISO7380_Pad_TopBottom
- S3: moved to B.Cu
- moved R4 7.75 mm to (124.2, 107.3), turned to 0 degrees
- moved S3 4.00 mm to (91.6, 104.0)
- moved R3 3.07 mm to (124.2, 105.0)
- moved R6 2.00 mm to (94.6, 107.7), turned to 180 degrees
- moved H3 0.40 mm to (93.6, 111.9)
- moved R5 0.10 mm to (93.6, 105.0)
Routing:
- net GND: track 12.1 -> 19.9 mm
Other:
- board size 5.9 x 12.7 mm -> 5.9 x 12.1 mm
