File: _QRE-Board_/QREBoard/QREBoard.kicad_sch (KiCad schematic)
At the start: 17 parts, among them J1 Conn_01x04_Pin, J2 Conn_01x03_Pin

Commit message: SOme changes
Parts:
- H3: footprint MountingHole:MountingHole_3.2mm_M3_ISO7380_Pad_TopBottom -> MountingHole:MountingHole_3.2mm_M3_ISO7380_Pad_TopOnly
Changed lines of the file:
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@@
 			)
 		)
-		(property "Footprint" "MountingHole:MountingHole_3.2mm_M3_ISO7380_Pad_TopBottom"
+		(property "Footprint" "MountingHole:MountingHole_3.2mm_M3_ISO7380_Pad_TopOnly"
 			(at 246.38 100.33 0)
 			(hide yes)
