File: _QRE-Boards_/QRE-Board_BackSen/QRE-Board_BackSen.kicad_sch (KiCad schematic)
At the start: 3 parts, among them U1 QRE1113GR

Commit message: Remove junk and regesign QRE-Boards
Parts:
- removed U1: QRE1113GR, OptoDevice:OnSemi_CASE100CY, symbol Sensor_Proximity:QRE1113GR
- added H1: M3, MountingHole:MountingHole_3.2mm_M3_Pad, symbol Mechanical:MountingHole_Pad
- added U1: QRE1113, OptoDevice:OnSemi_CASE100AQ, symbol Sensor_Proximity:QRE1113
Connections:
- net GND: now also H1.1, U1.2 (K), U1.4
- net QRE-Back: now also U1.3
- net at R1.2: now also U1.1 (A)
Other:
- note added: "Mount Hole"
- note added: "QRE1113GR"
- note added: "Senzor"
- company: (none) -> Maded by Vadim Sobčuk
- title: (none) -> Back QRE senzor for MiniSumo robot
- moved on the sheet: R1, R2
