File: _QRE-Boards_/QRE-Board_BackSen/QRE-Board_BackSen.kicad_pcb (KiCad board)
At the start: 2 copper layers, 5.9 x 11.3 mm, 4 parts, among them U1 QRE1113

Commit message: some changes
Other:
- board text added: "BTM"
Changed lines of the file:
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@@
 		(layer "Edge.Cuts")
+	)
+	(gr_text "BTM"
+		(at 151.25 108.5 0)
+		(layer "B.Cu")
+		(effects
+			(font
+				(size 1.25 1.25)
+				(bold yes)
+			)
+			(justify mirror)
+		)
 	)
 	(dimension
