File: _QRE-Boards_/QRE-Board_FrontSen/QRE-Board_FrontSen.kicad_pcb (KiCad board)
At the start: 2 copper layers, 94 x 18.3 mm, 12 parts, among them J1 Conn_01x04_Pin, U1 QRE1113GR, U2 QRE1113GR

Commit message: Remove junk and regesign QRE-Boards
Parts:
- renumbered TP1 to TPL1, TP2 to TPR1
Other:
- board text added: "Airsoftka was here"
